Commit message: Rename openarm_grip to openarm in moveit

File: openarm_moveit_config/config/openarm.ros2_control.xacro (robot description, xacro)
@@ -1,5 +1,5 @@
 <?xml version="1.0"?>
 <robot xmlns:xacro="http://www.ros.org/wiki/xacro">
-    <xacro:macro name="openarm_grip_ros2_control" params="name initial_positions_file">
+    <xacro:macro name="openarm_ros2_control" params="name initial_positions_file">
         <xacro:property name="initial_positions" value="${xacro.load_yaml(initial_positions_file)['initial_positions']}"/>
         <ros2_control name="${name}" type="system">

File: openarm_moveit_config/config/openarm.urdf.xacro (robot description, xacro)
@@ -1,9 +1,9 @@
 <?xml version="1.0"?>
-<robot xmlns:xacro="http://www.ros.org/wiki/xacro" name="openarm_grip">
+<robot xmlns:xacro="http://www.ros.org/wiki/xacro" name="openarm">
     <xacro:arg name="initial_positions_file" default="initial_positions.yaml" />
     <!-- Import openarm urdf file -->
     <xacro:include filename="$(find openarm_description)/urdf/openarm.urdf" />
     <!-- Import control_xacro -->
-    <xacro:include filename="openarm_grip.ros2_control.xacro" />
-    <xacro:openarm_grip_ros2_control name="FakeSystem" initial_positions_file="$(arg initial_positions_file)"/>
+    <xacro:include filename="openarm.ros2_control.xacro" />
+    <xacro:openarm_ros2_control name="FakeSystem" initial_positions_file="$(arg initial_positions_file)"/>
 </robot>

Commit message: Update moveit_config

File: openarm_moveit_config/config/openarm.ros2_control.xacro (robot description, xacro)
@@ -11,72 +11,80 @@
                 <command_interface name="position"/>
                 <command_interface name="velocity"/>
+                <command_interface name="effort"/>
                 <state_interface name="position">
                   <param name="initial_value">${initial_positions['rev1']}</param>
                 </state_interface>
                 <state_interface name="velocity"/>
+                <state_interface name="effort"/>
             </joint>
             <joint name="rev2">
                 <command_interface name="position"/>
                 <command_interface name="velocity"/>
+                <command_interface name="effort"/>
                 <state_interface name="position">
                   <param name="initial_value">${initial_positions['rev2']}</param>
                 </state_interface>
                 <state_interface name="velocity"/>
+                <state_interface name="effort"/>
             </joint>
             <joint name="rev3">
                 <command_interface name="position"/>
                 <command_interface name="velocity"/>
+                <command_interface name="effort"/>
                 <state_interface name="position">
                   <param name="initial_value">${initial_positions['rev3']}</param>
                 </state_interface>
                 <state_interface name="velocity"/>
+                <state_interface name="effort"/>
             </joint>
             <joint name="rev4">
                 <command_interface name="position"/>
                 <command_interface name="velocity"/>
+                <command_interface name="effort"/>
                 <state_interface name="position">
                   <param name="initial_value">${initial_positions['rev4']}</param>
                 </state_interface>
                 <state_interface name="velocity"/>
+                <state_interface name="effort"/>
             </joint>
             <joint name="rev5">
                 <command_interface name="position"/>
                 <command_interface name="velocity"/>
+                <command_interface name="effort"/>
                 <state_interface name="position">
                   <param name="initial_value">${initial_positions['rev5']}</param>
                 </state_interface>
                 <state_interface name="velocity"/>
+                <state_interface name="effort"/>
             </joint>
             <joint name="rev6">
                 <command_interface name="position"/>
                 <command_interface name="velocity"/>
+                <command_interface name="effort"/>
                 <state_interface name="position">
                   <param name="initial_value">${initial_positions['rev6']}</param>
                 </state_interface>
                 <state_interface name="velocity"/>
+                <state_interface name="effort"/>
             </joint>
             <joint name="rev7">
                 <command_interface name="position"/>
                 <command_interface name="velocity"/>
+                <command_interface name="effort"/>
                 <state_interface name="position">
                   <param name="initial_value">${initial_positions['rev7']}</param>
                 </state_interface>
                 <state_interface name="velocity"/>
+                <state_interface name="effort"/>
             </joint>
-            <joint name="slider_left">
+            <joint name="left_pris1">
                 <command_interface name="position"/>
                 <command_interface name="velocity"/>
+                <command_interface name="effort"/>
                 <state_interface name="position">
-                  <param name="initial_value">${initial_positions['slider_left']}</param>
+                  <param name="initial_value">${initial_positions['left_pris1']}</param>
                 </state_interface>
                 <state_interface name="velocity"/>
-            </joint>
-            <joint name="slider_right">
-                <command_interface name="position"/>
-                <command_interface name="velocity"/>
-                <state_interface name="position">
-                  <param name="initial_value">${initial_positions['slider_right']}</param>
-                </state_interface>
-                <state_interface name="velocity"/>
+                <state_interface name="effort"/>
             </joint>
         </ros2_control>

Commit message: Update openarm_moveit_config configs

File: openarm_moveit_config/config/openarm.ros2_control.xacro (robot description, xacro)
@@ -80,11 +80,13 @@
             <joint name="left_pris1">
                 <command_interface name="position"/>
-                <command_interface name="velocity"/>
-                <command_interface name="effort"/>
                 <state_interface name="position">
                   <param name="initial_value">${initial_positions['left_pris1']}</param>
                 </state_interface>
                 <state_interface name="velocity"/>
-                <state_interface name="effort"/>
+            </joint>
+            <joint name="left_pris1">
+                <state_interface name="position">
+                  <param name="initial_value">${initial_positions['left_pris1']}</param>
+                </state_interface>
             </joint>
         </ros2_control>
