Commit message: Update teleop

File: openarm_bimanual_description/urdf/openarm_bimanual.urdf (robot description, URDF)
Before this commit: robot openarm_bimanual, 22 links, 21 joints
Joints:
- joint left_fixed1: child right_link1 -> left_link1; origin xyz=-0.09 0.0 0.893 rpy=6.160245846096606 -1.5707963267948268 0.12293946108298068 -> xyz=0.09 0.0 0.893 rpy=3.0144791747751833 -1.5707963267948324 0.12689401604101067
- joint right_fixed1: child left_link1 -> right_link1; origin xyz=0.09 0.0 0.893 rpy=3.0144791747751833 -1.5707963267948324 0.12689401604101067 -> xyz=-0.09 0.0 0.893 rpy=6.160245846096606 -1.5707963267948268 0.12293946108298068

File: openarm_bimanual_description/urdf/openarm_bimanual.urdf.xacro (robot description, xacro)
@@ -4,6 +4,6 @@
   <xacro:include filename="$(find openarm_description)/urdf/openarm.xacro"/>
   <xacro:include filename="openarm_pedestal.urdf"/>
-  <xacro:openarm prefix="right_" side="right" zero_pos="arm"/>
-  <xacro:openarm prefix="left_" side="left" zero_pos="arm"/>
+  <xacro:openarm prefix="right_" side="right" zero_pos="arm" can_device="can0"/>
+  <xacro:openarm prefix="left_" side="left" zero_pos="arm" can_device="can1"/>
   <joint name="dummy_joint" type="fixed">
     <parent link="world"/>

File: openarm_description/urdf/openarm.ros2_control.xacro (robot description, xacro)
@@ -1,5 +1,5 @@
 <?xml version="1.0"?>
 <robot xmlns:xacro="http://www.ros.org/wiki/xacro">
-    <xacro:macro name="openarm_ros2_control" params="name initial_positions_file prefix:=''">
+    <xacro:macro name="openarm_ros2_control" params="name initial_positions_file prefix:='' can_device='can0'">
         <xacro:property name="initial_positions" value="${xacro.load_yaml(initial_positions_file)['initial_positions']}"/>
         <ros2_control name="${prefix}${name}" type="system">
@@ -8,4 +8,6 @@
                 <!-- <plugin>mock_components/GenericSystem</plugin> -->
                 <plugin>openarm_hardware/OpenArmHW</plugin>
+                <param name="prefix">${prefix}</param>
+                <param name="can_device">${can_device}</param>
             </hardware>
             <joint name="${prefix}rev1">
@@ -86,9 +88,9 @@
                 <state_interface name="velocity"/>
             </joint>
-            <joint name="${prefix}right_pris2">
+            <!-- <joint name="${prefix}right_pris2">
                 <state_interface name="position">
                   <param name="initial_value">${initial_positions['right_pris2']}</param>
                 </state_interface>
-            </joint>
+            </joint> -->
         </ros2_control>
     </xacro:macro>

File: openarm_description/urdf/openarm.urdf.xacro (robot description, xacro)
@@ -2,7 +2,5 @@
 <robot xmlns:xacro="http://www.ros.org/wiki/xacro" name="openarm">
     <xacro:include filename="openarm.xacro"/>
-    <xacro:openarm/>
-    <xacro:include filename="openarm_sensors.xacro"/>
-    <xacro:include filename="openarm.ros2_control.xacro" />
-    <xacro:openarm_ros2_control name="OpenArmHW" prefix="${prefix}" initial_positions_file="$(arg initial_positions_file)"/>
+    <xacro:openarm />
+    <xacro:include filename="$(find openarm_description)/urdf/openarm_sensors.xacro"/>
 </robot>

File: openarm_description/urdf/openarm.xacro (robot description, xacro)
@@ -4,5 +4,5 @@
         <color rgba="${105/255} ${105/255} ${105/255} 1.0"/>
     </material>
-    <xacro:macro name="openarm" params="side:='right' prefix:='' zero_pos='up'">
+    <xacro:macro name="openarm" params="side:='right' prefix:='' zero_pos='up' can_device='can0'">
         <!-- side right, left -->
         <!-- recommended prefixes left_, right_, etc. -->
@@ -10,5 +10,7 @@
         <xacro:property name="reflect" value="${1 if side=='right' else -1}"/>
         <xacro:property name="rotate" value="${0 if side=='right' else pi}"/>
-        <xacro:arg name="initial_positions_file" default="initial_positions.yaml" />
+        <xacro:include filename="$(find openarm_description)/urdf/openarm.ros2_control.xacro" />
+        <xacro:arg name="initial_positions_file" default="$(find openarm_description)/config/initial_positions.yaml" />
+        <xacro:openarm_ros2_control name="OpenArmHW" prefix="${prefix}" initial_positions_file="$(arg initial_positions_file)" can_device="${can_device}"/>
         <link name="${prefix}link1">
             <visual>

Commit message: Tweak urdfs and hardware interfaces to be representative of true rotation and gear ratios

File: openarm_bimanual_description/urdf/openarm_bimanual.urdf (robot description, URDF)
Before this commit: robot openarm_bimanual, 22 links, 21 joints
Links:
- removed link left_link1
- removed link left_link2
- removed link left_link3
- removed link left_link4
- removed link left_link5
- removed link left_link6
- removed link left_link7
- removed link left_link8
- removed link left_link_left_jaw
- removed link left_link_right_jaw
- added link camera_accel_frame
- added link camera_accel_optical_frame
- added link camera_bottom_screw_frame
- added link camera_color_frame
- added link camera_color_optical_frame
- added link camera_depth_frame
- added link camera_depth_optical_frame
- added link camera_gyro_frame
- added link camera_gyro_optical_frame
- added link camera_infra1_frame
- added link camera_infra1_optical_frame
- added link camera_infra2_frame
- added link camera_infra2_optical_frame
- added link camera_link, mass 0.072; collision box size=0.02505 0.09 0.025; visual mesh filename=file:///opt/ros/humble/share/realsense2_description/meshes/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
- added link right_dummy_link
Joints:
- removed joint left_fixed1
- removed joint left_left_pris1
- removed joint left_rev1
- removed joint left_rev2
- removed joint left_rev3
- removed joint left_rev4
- removed joint left_rev5
- removed joint left_rev6
- removed joint left_rev7
- removed joint left_right_pris2
- added joint camera_accel_joint: type fixed, parent camera_link, child camera_accel_frame, origin xyz=-0.01174 -0.00552 0.0051 rpy=0 0 0
- added joint camera_accel_optical_joint: type fixed, parent camera_accel_frame, child camera_accel_optical_frame, origin xyz=0 0 0 rpy=-1.5707963267948966 0 -1.5707963267948966
- added joint camera_color_joint: type fixed, parent camera_link, child camera_color_frame, origin xyz=0 0.015 0 rpy=0 0 0
- added joint camera_color_optical_joint: type fixed, parent camera_color_frame, child camera_color_optical_frame, origin xyz=0 0 0 rpy=-1.5707963267948966 0 -1.5707963267948966
- added joint camera_depth_joint: type fixed, parent camera_link, child camera_depth_frame, origin xyz=0 0 0 rpy=0 0 0
- added joint camera_depth_optical_joint: type fixed, parent camera_depth_frame, child camera_depth_optical_frame, origin xyz=0 0 0 rpy=-1.5707963267948966 0 -1.5707963267948966
- added joint camera_gyro_joint: type fixed, parent camera_link, child camera_gyro_frame, origin xyz=-0.01174 -0.00552 0.0051 rpy=0 0 0
- added joint camera_gyro_optical_joint: type fixed, parent camera_gyro_frame, child camera_gyro_optical_frame, origin xyz=0 0 0 rpy=-1.5707963267948966 0 -1.5707963267948966
- added joint camera_infra1_joint: type fixed, parent camera_link, child camera_infra1_frame, origin xyz=0 0.0 0 rpy=0 0 0
- added joint camera_infra1_optical_joint: type fixed, parent camera_infra1_frame, child camera_infra1_optical_frame, origin xyz=0 0 0 rpy=-1.5707963267948966 0 -1.5707963267948966
- added joint camera_infra2_joint: type fixed, parent camera_link, child camera_infra2_frame, origin xyz=0 -0.05 0 rpy=0 0 0
- added joint camera_infra2_optical_joint: type fixed, parent camera_infra2_frame, child camera_infra2_optical_frame, origin xyz=0 0 0 rpy=-1.5707963267948966 0 -1.5707963267948966
- added joint camera_joint: type fixed, parent pedestal_link, child camera_bottom_screw_frame, origin xyz=0.0 -0.025 0.995216 rpy=0.0 0.0 -1.5707963267948966
- added joint camera_link_joint: type fixed, parent camera_bottom_screw_frame, child camera_link, origin xyz=0.010600000000000002 0.0175 0.0125 rpy=0 0 0
- added joint right_dummy_joint: type fixed, parent right_dummy_link, child right_link1
- joint right_fixed1: child right_link1 -> right_dummy_link
- joint right_rev3: axis 0 0 1 -> 0 0 -1
- joint right_rev5: axis 0 0 1 -> 0 0 -1
- joint right_rev7: axis 0 0 1 -> 0 0 -1

File: openarm_description/urdf/openarm.xacro (robot description, xacro)
@@ -239,5 +239,5 @@
             <child link="${prefix}link4"/>
             <origin rpy="-1.5707963267949054 ${rotate} -1.562038143900564" xyz="-0.0612477 -0.000536432 0.02975"/>
-            <axis xyz="0 0 ${reflect*1}"/>
+            <axis xyz="0 0 -1"/>
             <limit effort="0.0" lower="-3.6651914291880923" upper="0.5235987755982988" velocity="0.0"/>
         </joint>
@@ -253,5 +253,5 @@
             <child link="${prefix}link6"/>
             <origin rpy="1.5707963267948473 -0.5569332500492129 1.556730325338251" xyz="-0.133937 0.00188408 -0.0297547"/>
-            <axis xyz="0 0 1"/>
+            <axis xyz="0 0 -1"/>
             <limit effort="0.0" lower="-2.0943951023931953" upper="2.0943951023931953" velocity="0.0"/>
         </joint>
@@ -267,5 +267,5 @@
             <child link="${prefix}link8"/>
             <origin rpy="-1.5707963267950005 -0.00875904933536772 -0.014066001454933467" xyz="-0.000217313 -0.0154485 0.0355"/>
-            <axis xyz="0 0 1"/>
+            <axis xyz="0 0 -1"/>
             <limit effort="0.0" lower="-0.9599310885968813" upper="0.9599310885968813" velocity="0.0"/>
         </joint>
@@ -275,5 +275,5 @@
             <origin rpy="1.570796326795101 -0.014066001454929162 0.00875904933542146" xyz="-0.1071 0.0768568 0.0132053"/>
             <axis xyz="0 0 1"/>
-            <limit effort="0.0" lower="0.0" upper="0.0451" velocity="0.0"/>
+            <limit effort="0.0" lower="-0.0451" upper="0.0" velocity="0.0"/>
         </joint>
         <joint name="${prefix}right_pris2" type="prismatic">
@@ -282,5 +282,5 @@
             <origin rpy="1.570796326794883 -0.014066001454927403 0.008759049336290027" xyz="-0.10571 -0.0781373 0.0132053"/>
             <axis xyz="0 0 1"/>
-            <limit effort="0.0" lower="0.0" upper="0.0451" velocity="0.0"/>
+            <limit effort="0.0" lower="-0.0451" upper="0.0" velocity="0.0"/>
             <mimic joint="${prefix}left_pris1" multiplier="-1.0" offset="0.0"/>
         </joint>

Commit message: Enable moveit2 for single and bimanual openarm

File: openarm_bimanual_description/urdf/openarm_bimanual.urdf (robot description, URDF)
Before this commit: robot openarm_bimanual, 27 links, 26 joints
Links:
- added link left_dummy_link
- added link left_link1, mass 0.5769283920617254; collision box size=0.11 0.073 0.0592; visual mesh filename=package://openarm_description/meshes/link1.stl
- added link left_link2, mass 0.16257504134917358; collision box size=0.0590000000149012 0.08200000000000002 0.0742471498637348; visual mesh filename=package://openarm_description/meshes/link2.stl
- added link left_link3, mass 0.4201676469910031; collision box size=0.08989101803441879 0.06999999999999983 0.05903276947803012; visual mesh filename=package://openarm_description/meshes/link3.stl
- added link left_link4, mass 0.819475539373447; collision box size=0.27584673777150337 0.08211429171582063 0.07186573179325861; visual mesh filename=package://openarm_description/meshes/link4.stl
- added link left_link5, mass 0.4086748254352304; collision box size=0.16827213220625828 0.06430555048399171 0.08257859967140947; visual mesh filename=package://openarm_description/meshes/link5.stl
- added link left_link6, mass 0.3448471958049249; collision box size=0.13114353004704765 0.05953478325301745 0.08817196195081879; visual mesh filename=package://openarm_description/meshes/link6_leftarm.stl
- added link left_link7, mass 0.2782138078738053; collision box size=0.058327402175132874 0.04432916698753661 0.08267601622411752; visual mesh filename=package://openarm_description/meshes/link7_leftarm.stl
- added link left_link8, mass 0.31261452743802165; collision box size=0.13038799671743653 0.05180887692688926 0.1601236763440867; visual mesh filename=package://openarm_description/meshes/link8.stl
- added link left_link_left_jaw, mass 0.04297897856394934; collision mesh filename=package://openarm_description/meshes/left_jaw.stl; visual mesh filename=package://openarm_description/meshes/left_jaw.stl
- added link left_link_right_jaw, mass 0.042981665301134515; collision mesh filename=package://openarm_description/meshes/right_jaw.stl; visual mesh filename=package://openarm_description/meshes/right_jaw.stl
Joints:
- added joint left_dummy_joint: type fixed, parent left_dummy_link, child left_link1
- added joint left_fixed1: type fixed, parent pedestal_link, child left_dummy_link, origin xyz=0.09 0.0 0.893 rpy=3.0144791747751833 -1.5707963267948324 0.12689401604101067
- added joint left_left_pris1: type prismatic, parent left_link8, child left_link_left_jaw, origin xyz=-0.1071 0.0768568 0.0132053 rpy=1.570796326795101 -0.014066001454929162 0.00875904933542146, axis 0 0 1, limit lower=-0.0451 upper=0.0 effort=0.0 velocity=0.0
- added joint left_rev1: type revolute, parent left_link1, child left_link2, origin xyz=0.0 0.0 0.05325 rpy=0 0 0, axis 0 0 -1, limit lower=-2.0943951023931953 upper=2.0943951023931953 effort=0.0 velocity=0.0
- added joint left_rev2: type revolute, parent left_link2, child left_link3, origin xyz=0.0 -0.02975 0.04475 rpy=-1.5707963267948968 0 0, axis 0 0 1, limit lower=0.0 upper=3.141592653589793 effort=0.0 velocity=0.0
- added joint left_rev3: type revolute, parent left_link3, child left_link4, origin xyz=-0.0612477 -0.000536432 0.02975 rpy=-1.5707963267949054 3.141592653589793 -1.562038143900564, axis 0 0 -1, limit lower=-3.6651914291880923 upper=0.5235987755982988 effort=0.0 velocity=0.0
- added joint left_rev4: type revolute, parent left_link4, child left_link5, origin xyz=0.0297547 0.0 -0.24175 rpy=-0.20701608758495998 -1.5707963267948566 -2.937419385117548, axis 0 0 1, limit lower=-0.3490658503988659 upper=2.792526803190927 effort=0.0 velocity=0.0
- added joint left_rev5: type revolute, parent left_link5, child left_link6, origin xyz=-0.133937 0.00188408 -0.0297547 rpy=1.5707963267948473 -0.5569332500492129 1.556730325338251, axis 0 0 -1, limit lower=-2.0943951023931953 upper=2.0943951023931953 effort=0.0 velocity=0.0
- added joint left_rev6: type revolute, parent left_link6, child left_link7, origin xyz=-0.0187648 -0.0301352 -0.12105 rpy=-1.5707963268024898 -1.5567303253382425 -0.5569332500461536, axis 0 0 1, limit lower=-1.5707963267948966 upper=1.5707963267948966 effort=0.0 velocity=0.0
- added joint left_rev7: type revolute, parent left_link7, child left_link8, origin xyz=-0.000217313 -0.0154485 0.0355 rpy=-1.5707963267950005 -0.00875904933536772 -0.014066001454933467, axis 0 0 -1, limit lower=-0.9599310885968813 upper=0.9599310885968813 effort=0.0 velocity=0.0
- added joint left_right_pris2: type prismatic, parent left_link8, child left_link_right_jaw, origin xyz=-0.10571 -0.0781373 0.0132053 rpy=1.570796326794883 -0.014066001454927403 0.008759049336290027, axis 0 0 1, limit lower=-0.0451 upper=0.0 effort=0.0 velocity=0.0, mimic joint=left_left_pris1 multiplier=-1.0 offset=0.0
- joint right_left_pris1: limit lower=0.0 upper=0.0451 effort=0.0 velocity=0.0 -> lower=-0.0451 upper=0.0 effort=0.0 velocity=0.0
- joint right_right_pris2: limit lower=0.0 upper=0.0451 effort=0.0 velocity=0.0 -> lower=-0.0451 upper=0.0 effort=0.0 velocity=0.0

File: openarm_bimanual_description/urdf/openarm_bimanual.urdf.xacro (robot description, xacro)
@@ -1,8 +1,8 @@
 <?xml version="1.0" ?>
 <robot xmlns:xacro="http://www.ros.org/wiki/xacro" name="openarm_bimanual">
-  <link name="world"/>
   <xacro:include filename="$(find openarm_description)/urdf/openarm.xacro"/>
   <xacro:include filename="openarm_pedestal.urdf"/>
   <xacro:include filename="openarm_bimanual_sensors.xacro"/>
+  <link name="world"/>
   <joint name="dummy_joint" type="fixed">
     <parent link="world"/>
@@ -10,10 +10,4 @@
     <origin xyz="0.0 0.0 0.0" rpy="0.0 0.0 0.0"/>
   </joint>
-  <!-- <xacro:openarm prefix="left_" side="left" zero_pos="arm" can_device="can1"/>
-  <joint name="left_fixed1" type="fixed">
-    <parent link="pedestal_link"/>
-    <child link="left_dummy_link"/>
-    <origin rpy="3.0144791747751833 -1.5707963267948324 0.12689401604101067" xyz="0.09 0.0 0.893"/>
-  </joint> -->
   <xacro:openarm prefix="right_" side="right" zero_pos="arm" can_device="can0"/>
   <joint name="right_fixed1" type="fixed">
@@ -22,3 +16,9 @@
     <origin rpy="${3.0186531925068127 + pi} -1.5707963267948268 0.12293946108298068" xyz="-0.09 0.0 0.893"/>
   </joint>
+  <xacro:openarm prefix="left_" side="left" zero_pos="arm" can_device="can1"/>
+  <joint name="left_fixed1" type="fixed">
+    <parent link="pedestal_link"/>
+    <child link="left_dummy_link"/>
+    <origin rpy="3.0144791747751833 -1.5707963267948324 0.12689401604101067" xyz="0.09 0.0 0.893"/>
+  </joint>
 </robot>

File: openarm_bimanual_moveit_config/config/openarm_bimanual.urdf.xacro (robot description, xacro)
@@ -4,6 +4,3 @@
     <!-- Import openarm_bimanual urdf file -->
     <xacro:include filename="$(find openarm_bimanual_description)/urdf/openarm_bimanual.urdf.xacro" />
-    <!-- Import control_xacro -->
-    <xacro:include filename="openarm_bimanual.ros2_control.xacro" />
-    <xacro:openarm_bimanual_ros2_control name="FakeSystem" initial_positions_file="$(arg initial_positions_file)"/>
 </robot>

File: openarm_description/urdf/openarm.ros2_control.xacro (robot description, xacro)
@@ -15,7 +15,5 @@
                 <command_interface name="velocity"/>
                 <command_interface name="effort"/>
-                <state_interface name="position">
-                  <param name="initial_value">${initial_positions['rev1']}</param>
-                </state_interface>
+                <state_interface name="position"/>
                 <state_interface name="velocity"/>
                 <state_interface name="effort"/>
@@ -25,7 +23,5 @@
                 <command_interface name="velocity"/>
                 <command_interface name="effort"/>
-                <state_interface name="position">
-                  <param name="initial_value">${initial_positions['rev2']}</param>
-                </state_interface>
+                <state_interface name="position"/>
                 <state_interface name="velocity"/>
                 <state_interface name="effort"/>
@@ -35,7 +31,5 @@
                 <command_interface name="velocity"/>
                 <command_interface name="effort"/>
-                <state_interface name="position">
-                  <param name="initial_value">${initial_positions['rev3']}</param>
-                </state_interface>
+                <state_interface name="position"/>
                 <state_interface name="velocity"/>
                 <state_interface name="effort"/>
@@ -45,7 +39,5 @@
                 <command_interface name="velocity"/>
                 <command_interface name="effort"/>
-                <state_interface name="position">
-                  <param name="initial_value">${initial_positions['rev4']}</param>
-                </state_interface>
+                <state_interface name="position"/>
                 <state_interface name="velocity"/>
                 <state_interface name="effort"/>
@@ -55,7 +47,5 @@
                 <command_interface name="velocity"/>
                 <command_interface name="effort"/>
-                <state_interface name="position">
-                  <param name="initial_value">${initial_positions['rev5']}</param>
-                </state_interface>
+                <state_interface name="position"/>
                 <state_interface name="velocity"/>
                 <state_interface name="effort"/>
@@ -65,7 +55,5 @@
                 <command_interface name="velocity"/>
                 <command_interface name="effort"/>
-                <state_interface name="position">
-                  <param name="initial_value">${initial_positions['rev6']}</param>
-                </state_interface>
+                <state_interface name="position"/>
                 <state_interface name="velocity"/>
                 <state_interface name="effort"/>
@@ -75,7 +63,5 @@
                 <command_interface name="velocity"/>
                 <command_interface name="effort"/>
-                <state_interface name="position">
-                  <param name="initial_value">${initial_positions['rev7']}</param>
-                </state_interface>
+                <state_interface name="position"/>
                 <state_interface name="velocity"/>
                 <state_interface name="effort"/>
@@ -83,7 +69,5 @@
             <joint name="${prefix}left_pris1">
                 <command_interface name="position"/>
-                <state_interface name="position">
-                  <param name="initial_value">${initial_positions['left_pris1']}</param>
-                </state_interface>
+                <state_interface name="position"/>
                 <state_interface name="velocity"/>
             </joint>

File: openarm_description/urdf/openarm.xacro (robot description, xacro)
@@ -225,5 +225,5 @@
             <child link="${prefix}link2"/>
             <origin rpy="0 0 0" xyz="0.0 0.0 0.05325"/>
-            <axis xyz="0 0 ${reflect*1}"/>
+            <axis xyz="0 0 1"/>
             <limit effort="0.0" lower="-2.0943951023931953" upper="2.0943951023931953" velocity="0.0"/>
         </joint>
@@ -232,5 +232,5 @@
             <child link="${prefix}link3"/>
             <origin rpy="-1.5707963267948968 ${pi/2 if zero_pos=='up' else 0} 0" xyz="0.0 -0.02975 0.04475"/>
-            <axis xyz="0 0 1"/>
+            <axis xyz="0 0 ${reflect * -1}"/>
             <limit effort="0.0" lower="${-pi/2.0 if zero_pos=='up' else 0.0}" upper="${pi/2 if zero_pos=='up' else pi}" velocity="0.0"/>
         </joint>
@@ -260,5 +260,5 @@
             <child link="${prefix}link7"/>
             <origin rpy="-1.5707963268024898 -1.5567303253382425 -0.5569332500461536" xyz="-0.0187648 -0.0301352 -0.12105"/>
-            <axis xyz="0 0 1"/>
+            <axis xyz="0 0 ${reflect}"/>
             <limit effort="0.0" lower="-1.5707963267948966" upper="1.5707963267948966" velocity="0.0"/>
         </joint>

File: openarm_moveit_config/config/openarm.urdf.xacro (robot description, xacro)
@@ -2,4 +2,4 @@
 <robot xmlns:xacro="http://www.ros.org/wiki/xacro" name="openarm">
     <!-- Import openarm urdf file -->
-    <xacro:include filename="$(find openarm_description)/urdf/openarm.urdf" />
+    <xacro:include filename="$(find openarm_description)/urdf/openarm.urdf.xacro" />
 </robot>
