Commit message: Marginally stable cotune

File: openarm_bimanual_description/urdf/openarm_bimanual.urdf (robot description, URDF)
Before this commit: robot openarm_bimanual, 40 links, 39 joints
Joints:
- removed joint left_left_pris1
- removed joint left_right_pris2
- removed joint right_left_pris1
- removed joint right_right_pris2
- added joint left_gripper: type prismatic, parent left_link8, child left_link_left_jaw, origin xyz=-0.1071 0.0768568 0.0132053 rpy=1.570796326795101 -0.014066001454929162 0.00875904933542146, axis 0 0 -1, limit lower=-0.0451 upper=0.0 effort=0.0 velocity=0.1
- added joint left_gripper_mimic: type prismatic, parent left_link8, child left_link_right_jaw, origin xyz=-0.10571 -0.0781373 0.0132053 rpy=1.570796326794883 -0.014066001454927403 0.008759049336290027, axis 0 0 -1, limit lower=-0.0451 upper=0.0 effort=0.0 velocity=0.0, mimic joint=left_gripper multiplier=-1.0 offset=0.0
- added joint right_gripper: type prismatic, parent right_link8, child right_link_left_jaw, origin xyz=-0.1071 0.0768568 0.0132053 rpy=1.570796326795101 -0.014066001454929162 0.00875904933542146, axis 0 0 -1, limit lower=-0.0451 upper=0.0 effort=0.0 velocity=0.1
- added joint right_gripper_mimic: type prismatic, parent right_link8, child right_link_right_jaw, origin xyz=-0.10571 -0.0781373 0.0132053 rpy=1.570796326794883 -0.014066001454927403 0.008759049336290027, axis 0 0 -1, limit lower=-0.0451 upper=0.0 effort=0.0 velocity=0.0, mimic joint=right_gripper multiplier=-1.0 offset=0.0

File: openarm_bimanual_moveit_config/config/openarm_bimanual.ros2_control.xacro (robot description, xacro)
@@ -132,17 +132,17 @@
                 <state_interface name="velocity"/>
             </joint>
-            <joint name="left_left_pris1">
+            <joint name="left_gripper">
                 <command_interface name="position"/>
                 <command_interface name="velocity"/>
                 <state_interface name="position">
-                  <param name="initial_value">${initial_positions['left_left_pris1']}</param>
+                  <param name="initial_value">${initial_positions['left_gripper']}</param>
                 </state_interface>
                 <state_interface name="velocity"/>
             </joint>
-            <joint name="right_left_pris1">
+            <joint name="right_gripper">
                 <command_interface name="position"/>
                 <command_interface name="velocity"/>
                 <state_interface name="position">
-                  <param name="initial_value">${initial_positions['right_left_pris1']}</param>
+                  <param name="initial_value">${initial_positions['right_gripper']}</param>
                 </state_interface>
                 <state_interface name="velocity"/>

File: openarm_description/urdf/openarm.robot.xacro (robot description, xacro)
@@ -25,4 +25,7 @@
         <xacro:property name="reflect" value="${1 if side=='right' else -1}"/>
         <xacro:property name="rotate" value="${0 if side=='right' else pi}"/>
+        <xacro:include filename="$(find openarm_description)/urdf/openarm.ros2_control.xacro" />
+        <xacro:arg name="initial_positions_file" default="$(find openarm_description)/config/initial_positions.yaml" />
+        <xacro:openarm_ros2_control name="OpenArmHW" prefix="${prefix}" initial_positions_file="$(arg initial_positions_file)" can_device="${can_device}" websocket_port="${1337 if side=='right' else 1338}"/>
         <link name="${prefix}dummy_link"/>
         <joint name="${prefix}dummy_joint" type="fixed">
@@ -280,5 +283,6 @@
             <limit effort="0.0" lower="${-pi * 11.0 / 36.0}" upper="${pi * 11.0 / 36.0}" velocity="0.0"/>
         </joint>
-        <joint name="${prefix}left_pris1" type="prismatic">
+        <!-- this is used as the actuator interface, the other gripper mimics motion -->
+        <joint name="${prefix}gripper" type="prismatic">
             <parent link="${prefix}link8"/>
             <child link="${prefix}link_left_jaw"/>
@@ -287,5 +291,5 @@
             <limit effort="0.0" lower="-0.0451" upper="0.0" velocity="0.1"/>
         </joint>
-        <joint name="${prefix}right_pris2" type="prismatic">
+        <joint name="${prefix}gripper_mimic" type="prismatic">
             <parent link="${prefix}link8"/>
             <child link="${prefix}link_right_jaw"/>
@@ -293,5 +297,5 @@
             <axis xyz="0 0 -1"/>
             <limit effort="0.0" lower="-0.0451" upper="0.0" velocity="0.0"/>
-            <mimic joint="${prefix}left_pris1" multiplier="-1.0" offset="0.0"/>
+            <mimic joint="${prefix}gripper" multiplier="-1.0" offset="0.0"/>
         </joint>
         <joint name="${prefix}virtual_gripper_center" type="fixed">

File: openarm_description/urdf/openarm.ros2_control.xacro (robot description, xacro)
@@ -86,9 +86,14 @@
                 <!-- <state_interface name="effort"/> -->
             </joint>
-            <joint name="${prefix}left_pris1">
+            <joint name="${prefix}gripper">
                 <command_interface name="position"/>
                 <state_interface name="position"/>
                 <state_interface name="velocity"/>
             </joint>
+            <!-- <joint name="${prefix}gripper_mimic">
+                <state_interface name="position">
+                  <param name="initial_value">${initial_positions['gripper_mimic']}</param>
+                </state_interface>
+            </joint> -->
         </ros2_control>
     </xacro:macro>

File: openarm_description/urdf/openarm.urdf (robot description, URDF)
Before this commit: robot openarm, 12 links, 11 joints
Joints:
- removed joint left_pris1
- removed joint right_pris2
- added joint gripper: type prismatic, parent link8, child link_left_jaw, origin xyz=-0.1071 0.0768568 0.0132053 rpy=1.570796326795101 -0.014066001454929162 0.00875904933542146, axis 0 0 -1, limit lower=-0.0451 upper=0.0 effort=0.0 velocity=0.1
- added joint gripper_mimic: type prismatic, parent link8, child link_right_jaw, origin xyz=-0.10571 -0.0781373 0.0132053 rpy=1.570796326794883 -0.014066001454927403 0.008759049336290027, axis 0 0 -1, limit lower=-0.0451 upper=0.0 effort=0.0 velocity=0.0, mimic joint=gripper multiplier=-1.0 offset=0.0
