Commit message: Add ego camera frame

File: openarm_bimanual_description/urdf/openarm_bimanual.urdf.xacro (robot description, xacro)
@@ -4,4 +4,5 @@
   <xacro:include filename="$(find openarm_description)/urdf/openarm.xacro"/>
   <xacro:include filename="openarm_pedestal.urdf"/>
+  <xacro:include filename="openarm_bimanual_sensors.xacro"/>
   <xacro:openarm prefix="right_" side="right" zero_pos="arm" can_device="can0"/>
   <xacro:openarm prefix="left_" side="left" zero_pos="arm" can_device="can1"/>

File: openarm_bimanual_description/urdf/openarm_bimanual_sensors.xacro (robot description, xacro)
@@ -1,3 +1,27 @@
 <?xml version="1.0"?>
 <robot xmlns:xacro="http://www.ros.org/wiki/xacro">
+    <link name="ego_camera_frame">
+        <visual>
+            <geometry>
+                <box size="0.09 0.025 0.025"/>
+            </geometry>
+            <material name="dark_gray"/>
+        </visual>
+        <collision>
+            <geometry>
+                <box size="0.09 0.025 0.025"/>
+            </geometry>
+        </collision>
+    </link>
+    <joint name="ego_camera_joint" type="fixed">
+        <parent link="pedestal_link"/>
+        <child link="ego_camera_frame"/>
+        <origin xyz="0.0 -0.025 0.995216" rpy="0.0 0.0 0.0"/>
+    </joint>
+    <link name="ego_camera_optical_frame"/>
+    <joint name="ego_camera_optical_joint" type="fixed">
+        <parent link="ego_camera_frame"/>
+        <child link="ego_camera_optical_frame"/>
+        <origin xyz="0.0 0.0 0.0" rpy="${pi/2.0} ${pi/2.0} 0.0"/>
+    </joint>
 </robot>

File: openarm_description/urdf/openarm.xacro (robot description, xacro)
@@ -3,4 +3,7 @@
     <material name="gray">
         <color rgba="${105/255} ${105/255} ${105/255} 1.0"/>
+    </material>
+    <material name="dark_gray">
+        <color rgba="${50/255} ${50/255} ${50/255} 1.0"/>
     </material>
     <xacro:macro name="openarm" params="side:='right' prefix:='' zero_pos='up' can_device='can0'">

Commit message: Update descriptions

File: openarm_bimanual_description/urdf/openarm_bimanual.urdf.xacro (robot description, xacro)
@@ -5,6 +5,4 @@
   <xacro:include filename="openarm_pedestal.urdf"/>
   <xacro:include filename="openarm_bimanual_sensors.xacro"/>
-  <xacro:openarm prefix="right_" side="right" zero_pos="arm" can_device="can0"/>
-  <xacro:openarm prefix="left_" side="left" zero_pos="arm" can_device="can1"/>
   <joint name="dummy_joint" type="fixed">
     <parent link="world"/>
@@ -12,12 +10,14 @@
     <origin xyz="0.0 0.0 0.0" rpy="0.0 0.0 0.0"/>
   </joint>
+  <!-- <xacro:openarm prefix="left_" side="left" zero_pos="arm" can_device="can1"/>
   <joint name="left_fixed1" type="fixed">
     <parent link="pedestal_link"/>
-    <child link="left_link1"/>
+    <child link="left_dummy_link"/>
     <origin rpy="3.0144791747751833 -1.5707963267948324 0.12689401604101067" xyz="0.09 0.0 0.893"/>
-  </joint>
+  </joint> -->
+  <xacro:openarm prefix="right_" side="right" zero_pos="arm" can_device="can0"/>
   <joint name="right_fixed1" type="fixed">
     <parent link="pedestal_link"/>
-    <child link="right_link1"/>
+    <child link="right_dummy_link"/>
     <origin rpy="${3.0186531925068127 + pi} -1.5707963267948268 0.12293946108298068" xyz="-0.09 0.0 0.893"/>
   </joint>

File: openarm_description/urdf/openarm.urdf (robot description, URDF)
Before this commit: robot openarm, 10 links, 9 joints
Links:
- added link dummy_link
Joints:
- added joint dummy_joint: type fixed, parent dummy_link, child link1

File: openarm_description/urdf/openarm.urdf.xacro (robot description, xacro)
@@ -2,5 +2,5 @@
 <robot xmlns:xacro="http://www.ros.org/wiki/xacro" name="openarm">
     <xacro:include filename="openarm.xacro"/>
-    <xacro:openarm />
+    <xacro:openarm/>
     <xacro:include filename="$(find openarm_description)/urdf/openarm_sensors.xacro"/>
 </robot>

File: openarm_description/urdf/openarm.xacro (robot description, xacro)
@@ -16,4 +16,9 @@
         <xacro:arg name="initial_positions_file" default="$(find openarm_description)/config/initial_positions.yaml" />
         <xacro:openarm_ros2_control name="OpenArmHW" prefix="${prefix}" initial_positions_file="$(arg initial_positions_file)" can_device="${can_device}"/>
+        <link name="${prefix}dummy_link"/>
+        <joint name="${prefix}dummy_joint" type="fixed">
+            <parent link="${prefix}dummy_link"/>
+            <child link="${prefix}link1"/>
+        </joint>
         <link name="${prefix}link1">
             <visual>

Commit message: Refactor to support three type of ros2_control hardware interfaces: real (physical openarm), sim (MuJoCo), mock (state follows commands)

File: openarm_bimanual_description/urdf/openarm_bimanual.urdf.xacro (robot description, xacro)
@@ -13,4 +13,5 @@
 -->
 <robot xmlns:xacro="http://www.ros.org/wiki/xacro" name="openarm_bimanual">
+  <xacro:arg name="hardware_type" default="real" />
   <!-- Robot description parameters -->
   <xacro:arg name="prefix" default="" />

File: openarm_bimanual_moveit_config/config/openarm_bimanual.urdf.xacro (robot description, xacro)
@@ -14,4 +14,5 @@
 <robot xmlns:xacro="http://www.ros.org/wiki/xacro" name="openarm_bimanual">
     <xacro:arg name="initial_positions_file" default="initial_positions.yaml" />
+    <xacro:arg name="hardware_type" default="real" />
     <!-- Import openarm_bimanual urdf file -->
     <xacro:include filename="$(find openarm_bimanual_description)/urdf/openarm_bimanual.urdf.xacro" />
@@ -22,6 +23,3 @@
         <origin xyz="0.0 0.0 0.0" rpy="0.0 0.0 0.0"/>
     </joint>
-    <!-- Import control_xacro -->
-    <!-- <xacro:include filename="openarm_bimanual.ros2_control.xacro" />
-    <xacro:openarm_bimanual_ros2_control name="FakeSystem" initial_positions_file="$(arg initial_positions_file)"/> -->
 </robot>

File: openarm_description/urdf/openarm.robot.xacro (robot description, xacro)
@@ -27,5 +27,5 @@
         <xacro:include filename="$(find openarm_description)/urdf/openarm.ros2_control.xacro" />
         <xacro:arg name="initial_positions_file" default="$(find openarm_description)/config/initial_positions.yaml" />
-        <xacro:openarm_ros2_control name="OpenArmHW" prefix="${prefix}" initial_positions_file="$(arg initial_positions_file)" can_device="${can_device}" websocket_port="${1337 if side=='right' else 1338}"/>
+        <xacro:openarm_ros2_control name="OpenArmHW" prefix="${prefix}" initial_positions_file="$(arg initial_positions_file)" can_device="${can_device}" websocket_port="${1337 if side=='right' else 1338}" hardware_type="${hardware_type}"/>
         <link name="${prefix}dummy_link"/>
         <joint name="${prefix}dummy_joint" type="fixed">

File: openarm_description/urdf/openarm.ros2_control.xacro (robot description, xacro)
@@ -13,20 +13,22 @@
 -->
 <robot xmlns:xacro="http://www.ros.org/wiki/xacro">
-    <xacro:macro name="openarm_ros2_control" params="name initial_positions_file websocket_port='' prefix:='' can_device='can0' use_mock_hardware='false' mock_sensor_commands='{}'">
+    <xacro:macro name="openarm_ros2_control" params="name initial_positions_file websocket_port='' prefix:='' can_device='can0' hardware_type='real' mock_sensor_commands='{}'">
         <xacro:property name="initial_positions" value="${xacro.load_yaml(initial_positions_file)['initial_positions']}"/>
         <ros2_control name="${prefix}${name}" type="system">
             <hardware>
-                <xacro:if value="${use_mock_hardware}">
+                <xacro:if value="${hardware_type == 'mock'}">
                     <plugin>mock_components/GenericSystem</plugin>
                     <param name="mock_sensor_commands">${mock_sensor_commands}</param>
                 </xacro:if>
-                <xacro:unless value="${use_mock_hardware}">
+                <xacro:if value="${hardware_type == 'sim'}">
+                    <plugin>openarm_mujoco_hardware/MujocoHardware</plugin>
+                    <param name="prefix">${prefix}</param>
+                    <param name="websocket_port">${websocket_port}</param>
+                </xacro:if>
+                <xacro:if value="${hardware_type == 'real'}">
                     <plugin>openarm_hardware/OpenArmHW</plugin>
                     <param name="prefix">${prefix}</param>
-                    <param name="websocket_port">${websocket_port}</param>
-                    <!-- <plugin>openarm_hardware/OpenArmHW</plugin>
-                    <param name="prefix">${prefix}</param>
-                    <param name="can_device">${can_device}</param> -->
-                </xacro:unless>
+                    <param name="can_device">${can_device}</param>
+                </xacro:if>
             </hardware>
             <joint name="${prefix}rev1">

Commit message: Update use_mock_hardware to hardware_type

File: openarm_bimanual_description/urdf/openarm_bimanual.urdf.xacro (robot description, xacro)
@@ -19,5 +19,5 @@
   <xacro:arg name="right_can_device" default="can0" />
   <xacro:arg name="left_can_device" default="can1" />
-  <xacro:arg name="use_mock_hardware" default="false" />
+  <xacro:arg name="hardware_type" default="real" />
   <xacro:arg name="mock_sensor_commands" default="false" />
   <xacro:include filename="$(find openarm_description)/urdf/openarm.robot.xacro"/>
@@ -46,5 +46,5 @@
   <xacro:arg name="right_initial_positions_file" default="$(find openarm_description)/config/initial_positions.yaml" />
   <xacro:arg name="left_initial_positions_file" default="$(find openarm_description)/config/initial_positions.yaml" />
-  <xacro:openarm_ros2_control name="RightOpenArmHW" prefix="right_" initial_positions_file="$(arg right_initial_positions_file)" can_device="$(arg right_can_device)" use_mock_hardware="$(arg use_mock_hardware)" mock_sensor_commands="$(arg mock_sensor_commands)"/>
-  <xacro:openarm_ros2_control name="LeftOpenArmHW" prefix="left_" initial_positions_file="$(arg left_initial_positions_file)" can_device="$(arg left_can_device)" use_mock_hardware="$(arg use_mock_hardware)" mock_sensor_commands="$(arg mock_sensor_commands)"/>
+  <xacro:openarm_ros2_control name="RightOpenArmHW" prefix="right_" initial_positions_file="$(arg right_initial_positions_file)" can_device="$(arg right_can_device)" hardware_type="$(arg hardware_type)" mock_sensor_commands="$(arg mock_sensor_commands)"/>
+  <xacro:openarm_ros2_control name="LeftOpenArmHW" prefix="left_" initial_positions_file="$(arg left_initial_positions_file)" can_device="$(arg left_can_device)" hardware_type="$(arg hardware_type)" mock_sensor_commands="$(arg mock_sensor_commands)"/>
 </robot>

File: openarm_description/urdf/openarm.robot.xacro (robot description, xacro)
@@ -25,7 +25,5 @@
         <xacro:property name="reflect" value="${1 if side=='right' else -1}"/>
         <xacro:property name="rotate" value="${0 if side=='right' else pi}"/>
-        <xacro:include filename="$(find openarm_description)/urdf/openarm.ros2_control.xacro" />
-        <xacro:arg name="initial_positions_file" default="$(find openarm_description)/config/initial_positions.yaml" />
-        <xacro:openarm_ros2_control name="OpenArmHW" prefix="${prefix}" initial_positions_file="$(arg initial_positions_file)" can_device="${can_device}" websocket_port="${1337 if side=='right' else 1338}" hardware_type="${hardware_type}"/>
+        <!-- ros2_control configuration is handled separately in openarm.urdf.xacro -->
         <link name="${prefix}dummy_link"/>
         <joint name="${prefix}dummy_joint" type="fixed">

File: openarm_description/urdf/openarm.ros2_control.xacro (robot description, xacro)
@@ -15,4 +15,11 @@
     <xacro:macro name="openarm_ros2_control" params="name initial_positions_file websocket_port='' prefix:='' can_device='can0' hardware_type='real' mock_sensor_commands='{}'">
         <xacro:property name="initial_positions" value="${xacro.load_yaml(initial_positions_file)['initial_positions']}"/>
+        <!-- Set default websocket ports based on prefix if not provided -->
+        <xacro:if value="${hardware_type == 'sim' and websocket_port == ''}">
+            <xacro:property name="computed_websocket_port" value="${'1337' if prefix == 'right_' or prefix == '' else '1338'}"/>
+        </xacro:if>
+        <xacro:unless value="${hardware_type == 'sim' and websocket_port == ''}">
+            <xacro:property name="computed_websocket_port" value="${websocket_port}"/>
+        </xacro:unless>
         <ros2_control name="${prefix}${name}" type="system">
             <hardware>
@@ -24,5 +31,7 @@
                     <plugin>openarm_mujoco_hardware/MujocoHardware</plugin>
                     <param name="prefix">${prefix}</param>
-                    <param name="websocket_port">${websocket_port}</param>
+                    <xacro:if value="${computed_websocket_port != ''}">
+                        <param name="websocket_port">${computed_websocket_port}</param>
+                    </xacro:if>
                 </xacro:if>
                 <xacro:if value="${hardware_type == 'real'}">

File: openarm_description/urdf/openarm.urdf.xacro (robot description, xacro)
@@ -19,5 +19,5 @@
     <!-- Control-related parameters -->
     <xacro:arg name="can_device" default="can0" />
-    <xacro:arg name="use_mock_hardware" default="false" />
+    <xacro:arg name="hardware_type" default="real" />
     <xacro:arg name="mock_sensor_commands" default="false" />
     <!-- Include robot description (without control parameters) -->
@@ -27,4 +27,4 @@
     <xacro:include filename="$(find openarm_description)/urdf/openarm.ros2_control.xacro"/>
     <xacro:arg name="initial_positions_file" default="$(find openarm_description)/config/initial_positions.yaml" />
-    <xacro:openarm_ros2_control name="OpenArmHW" prefix="$(arg prefix)" initial_positions_file="$(arg initial_positions_file)" can_device="$(arg can_device)" use_mock_hardware="$(arg use_mock_hardware)" mock_sensor_commands="$(arg mock_sensor_commands)"/>
+    <xacro:openarm_ros2_control name="OpenArmHW" prefix="$(arg prefix)" initial_positions_file="$(arg initial_positions_file)" can_device="$(arg can_device)" hardware_type="$(arg hardware_type)" mock_sensor_commands="$(arg mock_sensor_commands)"/>
 </robot>
