Commit message: Enable octomap perception

File: openarm_bimanual_moveit_config/config/openarm_bimanual.urdf.xacro (robot description, xacro)
@@ -4,4 +4,9 @@
     <!-- Import openarm_bimanual urdf file -->
     <xacro:include filename="$(find openarm_bimanual_description)/urdf/openarm_bimanual.urdf.xacro" />
+    <!-- <joint name="world_to_pedestal" type="fixed">
+        <parent link="world"/>
+        <child link="pedestal_link"/>
+        <origin xyz="0.0 0.0 0.0" rpy="0.0 0.0 0.0"/>
+    </joint> -->
     <!-- Import control_xacro -->
     <!-- <xacro:include filename="openarm_bimanual.ros2_control.xacro" />

Commit message: Fix base_link to world transform

File: openarm_bimanual_moveit_config/config/openarm_bimanual.urdf.xacro (robot description, xacro)
@@ -4,9 +4,10 @@
     <!-- Import openarm_bimanual urdf file -->
     <xacro:include filename="$(find openarm_bimanual_description)/urdf/openarm_bimanual.urdf.xacro" />
-    <!-- <joint name="world_to_pedestal" type="fixed">
+    <link name="base_link"/>
+    <joint name="world_to_pedestal" type="fixed">
         <parent link="world"/>
-        <child link="pedestal_link"/>
+        <child link="base_link"/>
         <origin xyz="0.0 0.0 0.0" rpy="0.0 0.0 0.0"/>
-    </joint> -->
+    </joint>
     <!-- Import control_xacro -->
     <!-- <xacro:include filename="openarm_bimanual.ros2_control.xacro" />
