Commit message: Correct right arm joint limits for rev2

File: openarm_description/urdf/openarm.xacro (robot description, xacro)
@@ -231,7 +231,7 @@
             <parent link="${prefix}link2"/>
             <child link="${prefix}link3"/>
-            <origin rpy="-1.5707963267948968 ${pi/2 if zero_pos=='up' else 0} 0" xyz="0.0 -0.02975 0.04475"/>
+            <origin rpy="-1.5707963267948968 ${pi/2 if zero_pos=='up' else 0.0} 0.0" xyz="0.0 -0.02975 0.04475"/>
             <axis xyz="0 0 ${reflect * -1}"/>
-            <limit effort="0.0" lower="${-pi/2.0 if zero_pos=='up' else 0.0}" upper="${pi/2 if zero_pos=='up' else pi}" velocity="0.0"/>
+            <limit effort="0.0" lower="${-pi/2.0 if zero_pos=='up' else -pi + rotate}" upper="${pi/2 if zero_pos=='up' else 0 + rotate}" velocity="0.0"/>
         </joint>
         <joint name="${prefix}rev3" type="revolute">

Commit message: Repair urdf to match physical robot

File: openarm_description/urdf/openarm.xacro (robot description, xacro)
@@ -241,5 +241,5 @@
             <origin rpy="-1.5707963267949054 ${rotate} -1.562038143900564" xyz="-0.0612477 -0.000536432 0.02975"/>
             <axis xyz="0 0 -1"/>
-            <limit effort="0.0" lower="-3.6651914291880923" upper="0.5235987755982988" velocity="0.0"/>
+            <limit effort="0.0" lower="${-0.52359 if side=='right' else -3.66519}" upper="${3.66519 if side=='right' else 0.52359}" velocity="0.0"/>
         </joint>
         <joint name="${prefix}rev4" type="revolute">
@@ -275,5 +275,5 @@
             <child link="${prefix}link_left_jaw"/>
             <origin rpy="1.570796326795101 -0.014066001454929162 0.00875904933542146" xyz="-0.1071 0.0768568 0.0132053"/>
-            <axis xyz="0 0 1"/>
+            <axis xyz="0 0 -1"/>
             <limit effort="0.0" lower="-0.0451" upper="0.0" velocity="0.0"/>
         </joint>
@@ -282,5 +282,5 @@
             <child link="${prefix}link_right_jaw"/>
             <origin rpy="1.570796326794883 -0.014066001454927403 0.008759049336290027" xyz="-0.10571 -0.0781373 0.0132053"/>
-            <axis xyz="0 0 1"/>
+            <axis xyz="0 0 -1"/>
             <limit effort="0.0" lower="-0.0451" upper="0.0" velocity="0.0"/>
             <mimic joint="${prefix}left_pris1" multiplier="-1.0" offset="0.0"/>

Commit message: Update openarm to support moveit2 bimanual planning with end effectors

File: openarm_description/urdf/openarm.xacro (robot description, xacro)
@@ -233,6 +233,6 @@
             <child link="${prefix}link3"/>
             <origin rpy="-1.5707963267948968 ${pi/2 if zero_pos=='up' else 0.0} 0.0" xyz="0.0 -0.02975 0.04475"/>
-            <axis xyz="0 0 ${reflect * -1}"/>
-            <limit effort="0.0" lower="${-pi/2.0 if zero_pos=='up' else -pi + rotate}" upper="${pi/2 if zero_pos=='up' else 0 + rotate}" velocity="0.0"/>
+            <axis xyz="0 0 1"/>
+            <limit effort="0.0" lower="${-pi/2.0 if zero_pos=='up' else 0}" upper="${pi/2 if zero_pos=='up' else pi}" velocity="0.0"/>
         </joint>
         <joint name="${prefix}rev3" type="revolute">
@@ -276,5 +276,5 @@
             <origin rpy="1.570796326795101 -0.014066001454929162 0.00875904933542146" xyz="-0.1071 0.0768568 0.0132053"/>
             <axis xyz="0 0 -1"/>
-            <limit effort="0.0" lower="-0.0451" upper="0.0" velocity="0.0"/>
+            <limit effort="0.0" lower="-0.0451" upper="0.0" velocity="0.1"/>
         </joint>
         <joint name="${prefix}right_pris2" type="prismatic">

Commit message: Fix rev1 to match hardware

File: openarm_description/urdf/openarm.xacro (robot description, xacro)
@@ -227,5 +227,5 @@
             <origin rpy="0 0 0" xyz="0.0 0.0 0.05325"/>
             <axis xyz="0 0 1"/>
-            <limit effort="0.0" lower="-2.0943951023931953" upper="2.0943951023931953" velocity="0.0"/>
+            <limit effort="0.0" lower="${-pi/4.0 if side=='right' and zero_pos=='arm' else -2.0943951023931953}" upper="${pi/4.0 if side=='left' and zero_pos=='arm' else 2.0943951023931953}" velocity="0.0"/>
         </joint>
         <joint name="${prefix}rev2" type="revolute">

Commit message: Align rev3 with hardware joint limits

File: openarm_description/urdf/openarm.xacro (robot description, xacro)
@@ -241,5 +241,5 @@
             <origin rpy="-1.5707963267949054 ${rotate} -1.562038143900564" xyz="-0.0612477 -0.000536432 0.02975"/>
             <axis xyz="0 0 -1"/>
-            <limit effort="0.0" lower="${-0.52359 if side=='right' else -3.66519}" upper="${3.66519 if side=='right' else 0.52359}" velocity="0.0"/>
+            <limit effort="0.0" lower="${-pi * 2.0 / 3.0}" upper="${pi * 2.0 / 3.0}" velocity="0.0"/>
         </joint>
         <joint name="${prefix}rev4" type="revolute">

Commit message: Match hardware joint limits

File: openarm_description/urdf/openarm.xacro (robot description, xacro)
@@ -234,5 +234,5 @@
             <origin rpy="-1.5707963267948968 ${pi/2 if zero_pos=='up' else 0.0} 0.0" xyz="0.0 -0.02975 0.04475"/>
             <axis xyz="0 0 1"/>
-            <limit effort="0.0" lower="${-pi/2.0 if zero_pos=='up' else 0}" upper="${pi/2 if zero_pos=='up' else pi}" velocity="0.0"/>
+            <limit effort="0.0" lower="${-pi/2.0 if zero_pos=='up' else -pi/18.0}" upper="${pi/2 if zero_pos=='up' else pi * 17.0 / 18.0}" velocity="0.0"/>
         </joint>
         <joint name="${prefix}rev3" type="revolute">
@@ -248,5 +248,5 @@
             <origin rpy="-0.20701608758495998 -1.5707963267948566 -2.937419385117548" xyz="0.0297547 0.0 -0.24175"/>
             <axis xyz="0 0 1"/>
-            <limit effort="0.0" lower="-0.3490658503988659" upper="2.792526803190927" velocity="0.0"/>
+            <limit effort="0.0" lower="0" upper="${pi * 5.0 / 6.0}" velocity="0.0"/>
         </joint>
         <joint name="${prefix}rev5" type="revolute">
@@ -255,5 +255,5 @@
             <origin rpy="1.5707963267948473 -0.5569332500492129 1.556730325338251" xyz="-0.133937 0.00188408 -0.0297547"/>
             <axis xyz="0 0 -1"/>
-            <limit effort="0.0" lower="-2.0943951023931953" upper="2.0943951023931953" velocity="0.0"/>
+            <limit effort="0.0" lower="${-pi * 2.0 / 3.0}" upper="${pi * 2.0 / 3.0}" velocity="0.0"/>
         </joint>
         <joint name="${prefix}rev6" type="revolute">
@@ -262,5 +262,5 @@
             <origin rpy="-1.5707963268024898 -1.5567303253382425 -0.5569332500461536" xyz="-0.0187648 -0.0301352 -0.12105"/>
             <axis xyz="0 0 ${reflect}"/>
-            <limit effort="0.0" lower="-1.5707963267948966" upper="1.5707963267948966" velocity="0.0"/>
+            <limit effort="0.0" lower="${-pi / 2.0}" upper="${pi / 2.0}" velocity="0.0"/>
         </joint>
         <joint name="${prefix}rev7" type="revolute">
@@ -269,5 +269,5 @@
             <origin rpy="-1.5707963267950005 -0.00875904933536772 -0.014066001454933467" xyz="-0.000217313 -0.0154485 0.0355"/>
             <axis xyz="0 0 -1"/>
-            <limit effort="0.0" lower="-0.9599310885968813" upper="0.9599310885968813" velocity="0.0"/>
+            <limit effort="0.0" lower="${-pi * 11.0 / 36.0}" upper="${pi * 11.0 / 36.0}" velocity="0.0"/>
         </joint>
         <joint name="${prefix}left_pris1" type="prismatic">
