Commit message: Add control interfaces to openarm_description

File: openarm_description/urdf/openarm.ros2_control.xacro (robot description, xacro)
@@ -1,5 +1,5 @@
 <?xml version="1.0"?>
 <robot xmlns:xacro="http://www.ros.org/wiki/xacro">
-    <xacro:macro name="openarm_ros2_control" params="name initial_positions_file">
+    <xacro:macro name="openarm_ros2_control" params="name initial_positions_file prefix:=''">
         <xacro:property name="initial_positions" value="${xacro.load_yaml(initial_positions_file)['initial_positions']}"/>
         <ros2_control name="${name}" type="system">
@@ -8,5 +8,5 @@
                 <plugin>mock_components/GenericSystem</plugin>
             </hardware>
-            <joint name="rev1">
+            <joint name="${prefix}rev1">
                 <command_interface name="position"/>
                 <command_interface name="velocity"/>
@@ -18,5 +18,5 @@
                 <state_interface name="effort"/>
             </joint>
-            <joint name="rev2">
+            <joint name="${prefix}rev2">
                 <command_interface name="position"/>
                 <command_interface name="velocity"/>
@@ -28,5 +28,5 @@
                 <state_interface name="effort"/>
             </joint>
-            <joint name="rev3">
+            <joint name="${prefix}rev3">
                 <command_interface name="position"/>
                 <command_interface name="velocity"/>
@@ -38,5 +38,5 @@
                 <state_interface name="effort"/>
             </joint>
-            <joint name="rev4">
+            <joint name="${prefix}rev4">
                 <command_interface name="position"/>
                 <command_interface name="velocity"/>
@@ -48,5 +48,5 @@
                 <state_interface name="effort"/>
             </joint>
-            <joint name="rev5">
+            <joint name="${prefix}rev5">
                 <command_interface name="position"/>
                 <command_interface name="velocity"/>
@@ -58,5 +58,5 @@
                 <state_interface name="effort"/>
             </joint>
-            <joint name="rev6">
+            <joint name="${prefix}rev6">
                 <command_interface name="position"/>
                 <command_interface name="velocity"/>
@@ -68,5 +68,5 @@
                 <state_interface name="effort"/>
             </joint>
-            <joint name="rev7">
+            <joint name="${prefix}rev7">
                 <command_interface name="position"/>
                 <command_interface name="velocity"/>
@@ -78,5 +78,5 @@
                 <state_interface name="effort"/>
             </joint>
-            <joint name="left_pris1">
+            <joint name="${prefix}left_pris1">
                 <command_interface name="position"/>
                 <state_interface name="position">
@@ -85,5 +85,5 @@
                 <state_interface name="velocity"/>
             </joint>
-            <joint name="left_pris1">
+            <joint name="${prefix}right_pris2">
                 <state_interface name="position">
                   <param name="initial_value">${initial_positions['left_pris1']}</param>

File: openarm_description/urdf/openarm.urdf.xacro (robot description, xacro)
@@ -3,4 +3,3 @@
     <xacro:include filename="openarm.xacro"/>
     <xacro:openarm/>
-    <xacro:include filename="openarm_sensors.urdf.xacro"/>
 </robot>

File: openarm_description/urdf/openarm.xacro (robot description, xacro)
@@ -10,4 +10,8 @@
         <xacro:property name="reflect" value="${1 if side=='right' else -1}"/>
         <xacro:property name="rotate" value="${0 if side=='right' else pi}"/>
+        <xacro:include filename="openarm_sensors.urdf.xacro"/>
+        <xacro:arg name="initial_positions_file" default="initial_positions.yaml" />
+        <xacro:include filename="openarm.ros2_control.xacro" />
+        <xacro:openarm_ros2_control name="openarm_control" prefix="${prefix}" initial_positions_file="$(arg initial_positions_file)"/>
         <link name="${prefix}link1">
             <visual>

File: openarm_moveit_config/config/openarm.urdf.xacro (robot description, xacro)
@@ -1,9 +1,5 @@
 <?xml version="1.0"?>
 <robot xmlns:xacro="http://www.ros.org/wiki/xacro" name="openarm">
-    <xacro:arg name="initial_positions_file" default="initial_positions.yaml" />
     <!-- Import openarm urdf file -->
     <xacro:include filename="$(find openarm_description)/urdf/openarm.urdf" />
-    <!-- Import control_xacro -->
-    <xacro:include filename="openarm.ros2_control.xacro" />
-    <xacro:openarm_ros2_control name="FakeSystem" initial_positions_file="$(arg initial_positions_file)"/>
 </robot>

Commit message: Partial arm working

File: openarm_description/urdf/openarm.ros2_control.xacro (robot description, xacro)
@@ -13,5 +13,5 @@
 -->
 <robot xmlns:xacro="http://www.ros.org/wiki/xacro">
-    <xacro:macro name="openarm_ros2_control" params="name initial_positions_file prefix:='' can_device='can0' use_mock_hardware:=false mock_sensor_commands:=false">
+    <xacro:macro name="openarm_ros2_control" params="name initial_positions_file websocket_port='' prefix:='' can_device='can0' use_mock_hardware='false' mock_sensor_commands='{}'">
         <xacro:property name="initial_positions" value="${xacro.load_yaml(initial_positions_file)['initial_positions']}"/>
         <ros2_control name="${prefix}${name}" type="system">
@@ -24,5 +24,8 @@
                     <plugin>openarm_hardware/OpenArmHW</plugin>
                     <param name="prefix">${prefix}</param>
-                    <param name="can_device">${can_device}</param>
+                    <param name="websocket_port">${websocket_port}</param>
+                    <!-- <plugin>openarm_hardware/OpenArmHW</plugin>
+                    <param name="prefix">${prefix}</param>
+                    <param name="can_device">${can_device}</param> -->
                 </xacro:unless>
             </hardware>
